File: Duet-0.8/Processor.sch (KiCad schematic (older format))
At the start: 42 parts, among them J21 JTAG, J26 GND, U1 ATSAM3X8E, X2 CRYSTAL_4PIN

Commit message: USB B connector used.  Always-on fan connector added next to heater connector. Green power LED (5v) now has a bigger ballast resistor.
Parts:
- removed J21: JTAG, symbol CONN_JTAG
Connections:
- wire segments 164 -> 154
Changed lines of the file:
@@
 Sheet 7 7
 Title "Duet"
-Date "18 mar 2015"
+Date "8 jul 2015"
 Rev "0.7"
 Comp "Think3DPrint3D, RepRapPro"
@@
 	7600 8900 9400 8900
 Connection ~ 9150 8900
-Connection ~ 9400 9500
-Wire Wire Line
-	9400 9400 9400 9500
+Wire Wire Line
+	9400 9400 9400 9850
 Connection ~ 10300 4150
 Wire Wire Line
@@
 	12250 4750 12250 4600
 Wire Wire Line
-	9800 9550 9500 9550
-Wire Wire Line
-	9500 9550 9500 9800
-Wire Wire Line
-	9500 9800 8600 9800
-Wire Wire Line
-	9800 9400 9650 9400
-Wire Wire Line
-	9650 9400 9650 9600
-Wire Wire Line
-	9650 9600 8600 9600
-Wire Wire Line
-	9800 9700 8600 9700
+	9550 9400 9800 9400
 Wire Wire Line
 	13200 14450 13400 14450
@@
 Wire Wire Line
 	8650 6400 8650 6200
-Connection ~ 7550 9900
-Wire Wire Line
-	7550 9950 7550 9600
-Wire Wire Line
-	7600 9700 7550 9700
-Wire Wire Line
-	7550 9600 7600 9600
-Wire Wire Line
-	8650 10100 8650 9900
 Wire Wire Line
 	8250 6400 8250 6600
 Connection ~ 8250 6400
 Wire Wire Line
-	7550 9900 7600 9900
-Connection ~ 7550 9700
-Wire Wire Line
 	10550 15500 10550 15150
 Wire Wire Line
@@
 Wire Wire Line
 	8650 5550 9800 5550
-Wire Wire Line
-	8600 9500 9550 9500
-Wire Wire Line
-	9550 9500 9550 9850
-Wire Wire Line
-	9550 9850 9800 9850
-Wire Wire Line
-	8650 10100 8600 10100
 Wire Wire Line
 	12100 4750 12100 4600
@@
 Wire Wire Line
 	8650 9400 8650 9800
-Connection ~ 8650 9800
 Wire Wire Line
 	9150 9400 9150 9600
-Connection ~ 9150 9600
 Wire Wire Line
 	9400 8900 9400 9000
@@
 Wire Wire Line
 	8650 8900 8650 9000
-Wire Wire Line
-	7600 9500 7600 8800
 Connection ~ 7600 8900
 Wire Wire Line
@@
 Wire Wire Line
 	15000 13850 15000 13650
-Wire Wire Line
-	8650 9900 8600 9900
 Wire Wire Line
 	11700 15450 11700 15500
@@
 $EndComp
 $Comp
-L GND #PWR056
+L GND #PWR057
 U 1 1 50F1BF81
 P 9200 14550
-F 0 "#PWR056" H 9200 14550 30  0001 C CNN
+F 0 "#PWR057" H 9200 14550 30  0001 C CNN
 F 1 "GND" H 9200 14480 30  0001 C CNN
 F 2 "" H 9200 14550 60  0001 C CNN
@@
 $EndComp
 $Comp
-L GND #PWR057
+L GND #PWR058
 U 1 1 50F1B3A2
 P 6500 5100
-F 0 "#PWR057" H 6500 5100 30  0001 C CNN
+F 0 "#PWR058" H 6500 5100 30  0001 C CNN
 F 1 "GND" H 6500 5030 30  0001 C CNN
 F 2 "" H 6500 5100 60  0001 C CNN
@@
 VDDPLL
 $Comp
-L GND #PWR058
+L GND #PWR059
 U 1 1 50F1AE7F
 P 12350 4000
-F 0 "#PWR058" H 12350 4000 30  0001 C CNN
+F 0 "#PWR059" H 12350 4000 30  0001 C CNN
 F 1 "GND" H 12350 3930 30  0001 C CNN
 F 2 "" H 12350 4000 60  0001 C CNN
@@
 $EndComp
 $Comp
-L GND #PWR059
+L GND #PWR060
 U 1 1 50F1AB2F
 P 13850 4500
-F 0 "#PWR059" H 13850 4500 30  0001 C CNN
+F 0 "#PWR060" H 13850 4500 30  0001 C CNN
 F 1 "GND" H 13850 4430 30  0001 C CNN
 F 2 "" H 13850 4500 60  0001 C CNN
@@
 $EndComp
 NoConn ~ 13200 14300
-Text GLabel 8600 10100 0    60   BiDi ~ 0
-RESET
 Text GLabel 13200 14750 2    60   BiDi ~ 0
 NRST
@@
 NoConn ~ 7600 9800
 $Comp
-L GND #PWR060
+L GND #PWR061
 U 1 1 50F13953
 P 13400 14500
-F 0 "#PWR060" H 13400 14500 30  0001 C CNN
+F 0 "#PWR061" H 13400 14500 30  0001 C CNN
 F 1 "GND" H 13400 14430 30  0001 C CNN
 F 2 "" H 13400 14500 60  0001 C CNN
@@
 $EndComp
 $Comp
-L GND #PWR061
+L GND #PWR062
 U 1 1 50F1392E
 P 13400 13750
-F 0 "#PWR061" H 13400 13750 30  0001 C CNN
+F 0 "#PWR062" H 13400 13750 30  0001 C CNN
 F 1 "GND" H 13400 13680 30  0001 C CNN
 F 2 "" H 13400 13750 60  0001 C CNN
@@
 $EndComp
 $Comp
-L CONN_JTAG J21
-U 1 1 505F8BB9
-P 8100 9700
-F 0 "J21" H 8100 9400 50  0000 C CNN
-F 1 "JTAG" H 8100 10000 35  0000 C CNN
-F 2 "" H 8100 9700 60  0001 C CNN
-F 3 "" H 8100 9700 60  0001 C CNN
-	1    8100 9700
-	1    0    0    -1
-$EndComp
-$Comp
-L GND #PWR062
+L GND #PWR063
 U 1 1 505DBB16
 P 11050 15700
-F 0 "#PWR062" H 11050 15700 30  0001 C CNN
+F 0 "#PWR063" H 11050 15700 30  0001 C CNN
 F 1 "GND" H 11050 15630 30  0001 C CNN
 F 2 "" H 11050 15700 60  0001 C CNN
@@
 SPI0_SPCK
 $Comp
-L GND #PWR063
+L GND #PWR064
 U 1 1 5057A432
 P 14800 14850
-F 0 "#PWR063" H 14800 14850 30  0001 C CNN
+F 0 "#PWR064" H 14800 14850 30  0001 C CNN
 F 1 "GND" H 14800 14780 30  0001 C CNN
 F 2 "" H 14800 14850 60  0001 C CNN
 F 3 "" H 14800 14850 60  0001 C CNN
 	1    14800 14850
-	1    0    0    -1
-$EndComp
-$Comp
-L GND #PWR064
-U 1 1 50579E73
-P 7550 9950
-F 0 "#PWR064" H 7550 9950 30  0001 C CNN
-F 1 "GND" H 7550 9880 30  0001 C CNN
-F 2 "" H 7550 9950 60  0001 C CNN
-F 3 "" H 7550 9950 60  0001 C CNN
-	1    7550 9950
 	1    0    0    -1
 $EndComp
@@
 	14750 6900 14750 7000
 Connection ~ 14800 6900
+Wire Wire Line
+	7600 8800 7600 8900
+Wire Wire Line
+	8650 9800 9700 9800
+Wire Wire Line
+	9800 9550 9700 9550
+Wire Wire Line
+	9400 9850 9800 9850
+Wire Wire Line
+	9700 9550 9700 9800
+Wire Wire Line
+	9550 9400 9550 9600
+Wire Wire Line
+	9550 9600 9150 9600
 $EndSCHEMATC

Commit message: Erase and Reset buttons replaced by jumpers.
Parts:
- removed S1: RESET, symbol SW_TACT
- removed S2: MCU ERASE, symbol SW_TACT
Connections:
- net labels added: ERASE
- wire segments 154 -> 137
Changed lines of the file:
@@
 Wire Wire Line
 	15000 13250 15000 13450
-Connection ~ 14800 14700
-Wire Wire Line
-	14800 14850 14800 14700
-Connection ~ 14800 14000
 Connection ~ 14800 13850
 Wire Wire Line
-	14800 13850 14800 14100
-Connection ~ 14800 7000
-Wire Wire Line
-	14800 6800 14800 7000
-Connection ~ 14800 7550
-Wire Wire Line
-	14800 7550 14800 7600
-Wire Wire Line
-	14800 7600 13200 7600
+	13200 7600 15150 7600
 Connection ~ 9250 14000
 Wire Wire Line
@@
 Wire Wire Line
 	9800 14000 9050 14000
-Wire Wire Line
-	14750 7500 14750 7550
-Wire Wire Line
-	14750 7550 14850 7550
-Wire Wire Line
-	14850 7550 14850 7500
-Wire Wire Line
-	14850 7000 14750 7000
-Wire Wire Line
-	14750 14600 14750 14700
-Wire Wire Line
-	14750 14700 14850 14700
-Wire Wire Line
-	14850 14700 14850 14600
 Wire Wire Line
 	15000 13850 15000 13650
@@
 MCDA1
 $Comp
-L SW_TACT S2
-U 1 1 50F1C331
-P 14800 7250
-F 0 "S2" H 14950 7100 60  0000 C CNN
-F 1 "MCU ERASE" H 14800 7450 60  0000 C CNN
-F 2 "" H 14800 7250 60  0001 C CNN
-F 3 "" H 14800 7250 60  0001 C CNN
-	1    14800 7250
-	0    -1   -1   0
-$EndComp
-Text GLabel 14800 6800 1    60   Input ~ 0
-+3.3V
-$Comp
 L C_SMALL C65
 U 1 1 50F1BFA1
@@
 $EndComp
 $Comp
-L GND #PWR057
+L GND #PWR058
 U 1 1 50F1BF81
 P 9200 14550
-F 0 "#PWR057" H 9200 14550 30  0001 C CNN
+F 0 "#PWR058" H 9200 14550 30  0001 C CNN
 F 1 "GND" H 9200 14480 30  0001 C CNN
 F 2 "" H 9200 14550 60  0001 C CNN
@@
 $EndComp
 $Comp
-L GND #PWR058
+L GND #PWR059
 U 1 1 50F1B3A2
 P 6500 5100
-F 0 "#PWR058" H 6500 5100 30  0001 C CNN
+F 0 "#PWR059" H 6500 5100 30  0001 C CNN
 F 1 "GND" H 6500 5030 30  0001 C CNN
 F 2 "" H 6500 5100 60  0001 C CNN
@@
 VDDPLL
 $Comp
-L GND #PWR059
+L GND #PWR060
 U 1 1 50F1AE7F
 P 12350 4000
-F 0 "#PWR059" H 12350 4000 30  0001 C CNN
+F 0 "#PWR060" H 12350 4000 30  0001 C CNN
 F 1 "GND" H 12350 3930 30  0001 C CNN
 F 2 "" H 12350 4000 60  0001 C CNN
@@
 $EndComp
 $Comp
-L GND #PWR060
+L GND #PWR061
 U 1 1 50F1AB2F
 P 13850 4500
-F 0 "#PWR060" H 13850 4500 30  0001 C CNN
+F 0 "#PWR061" H 13850 4500 30  0001 C CNN
 F 1 "GND" H 13850 4430 30  0001 C CNN
 F 2 "" H 13850 4500 60  0001 C CNN
@@
 NoConn ~ 7600 9800
 $Comp
-L GND #PWR061
+L GND #PWR062
 U 1 1 50F13953
 P 13400 14500
-F 0 "#PWR061" H 13400 14500 30  0001 C CNN
+F 0 "#PWR062" H 13400 14500 30  0001 C CNN
 F 1 "GND" H 13400 14430 30  0001 C CNN
 F 2 "" H 13400 14500 60  0001 C CNN
@@
 $EndComp
 $Comp
-L GND #PWR062
+L GND #PWR063
 U 1 1 50F1392E
 P 13400 13750
-F 0 "#PWR062" H 13400 13750 30  0001 C CNN
+F 0 "#PWR063" H 13400 13750 30  0001 C CNN
 F 1 "GND" H 13400 13680 30  0001 C CNN
 F 2 "" H 13400 13750 60  0001 C CNN
@@
 $EndComp
 $Comp
-L SW_TACT S1
-U 1 1 5075E99F
-P 14800 14350
-F 0 "S1" H 14950 14200 60  0000 C CNN
-F 1 "RESET" H 14800 14550 60  0000 C CNN
-F 2 "" H 14800 14350 60  0001 C CNN
-F 3 "" H 14800 14350 60  0001 C CNN
-	1    14800 14350
-	0    -1   -1   0
-$EndComp
-$Comp
 L C_SMALL C45
 U 1 1 50657171
@@
 $EndComp
 $Comp
-L GND #PWR063
+L GND #PWR064
 U 1 1 505DBB16
 P 11050 15700
-F 0 "#PWR063" H 11050 15700 30  0001 C CNN
+F 0 "#PWR064" H 11050 15700 30  0001 C CNN
 F 1 "GND" H 11050 15630 30  0001 C CNN
 F 2 "" H 11050 15700 60  0001 C CNN
@@
 Text GLabel 13200 10150 2    50   BiDi ~ 0
 SPI0_SPCK
-$Comp
-L GND #PWR064
-U 1 1 5057A432
-P 14800 14850
-F 0 "#PWR064" H 14800 14850 30  0001 C CNN
-F 1 "GND" H 14800 14780 30  0001 C CNN
-F 2 "" H 14800 14850 60  0001 C CNN
-F 3 "" H 14800 14850 60  0001 C CNN
-	1    14800 14850
-	1    0    0    -1
-$EndComp
 Text GLabel 11000 3900 1    60   Input ~ 0
 +3.3V
@@
 $EndComp
 Wire Wire Line
-	14750 14000 14850 14000
-Wire Wire Line
-	14850 14000 14850 14100
-Wire Wire Line
-	14750 14000 14750 14100
-Wire Wire Line
-	14850 7000 14850 6900
-Wire Wire Line
-	14850 6900 14750 6900
-Wire Wire Line
-	14750 6900 14750 7000
-Connection ~ 14800 6900
-Wire Wire Line
 	7600 8800 7600 8900
 Wire Wire Line
@@
 Wire Wire Line
 	9550 9600 9150 9600
+Text GLabel 15150 7600 2    60   BiDi ~ 0
+ERASE
 $EndSCHEMATC
